File: noise_gate/noise_gate.kicad_pcb (KiCad board)
At the start: 2 copper layers, 80 x 100 mm, 76 parts, among them J1 Jack_6.35, J2 Jack_6.35, J6 top_panel_connector, J7 Conn_01x01_Socket, J8 Conn_01x01_Socket, J9 Barrel_Jack_Switch, P1 front_panel, P2 bottom_panel, Q1 MMBT5551, Q10 AO3401A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

Commit message: White pcbs.
Parts:
- removed BT1: Battery_Cell, pedale:BatteryHolder_Eagle_12BH611-GR
- removed J7, J8: Conn_01x01_Socket, TestPoint:TestPoint_THTPad_D2.5mm_Drill1.2mm
- removed Q12: AO3400A, Package_TO_SOT_SMD:SOT-23
- removed Q6: AO3401A, Package_TO_SOT_SMD:SOT-23
- removed R23, R27: 100k, Resistor_SMD:R_0603_1608Metric_Pad0.98x0.95mm_HandSolder
- added J3: Jack_6.35, pedale:Jack_6.35mm, F.Cu at (67.2, 119.9)
- added J4: Jack_6.35, pedale:Jack_6.35mm, F.Cu at (112.8, 103.6)
- moved J2 6.50 mm to (67.2, 139.6)
- moved J1 6.50 mm to (112.8, 123.4)
Connections:
- J1 pad SN: IN_CONNECT -> unconnected-(J1-PadSN)
Routing:
- net IN_CONNECT: track 109.6 -> 0.00 mm, vias 2 -> 0
- net unconnected-(J3-PadTN): track 0.00 -> 53.5 mm, vias 0 -> 2
- net (no net): track 0.00 -> 33.3 mm
- net BAT+: track 28.7 -> 0.00 mm
- net Net-(Q12-D): track 4.61 -> 0.00 mm
