File: noise_gate/noise_gate.kicad_sch (KiCad schematic)
At the start: 76 parts, among them J1 Jack_6.35, J2 Jack_6.35, J6 top_panel_connector, J7 Conn_01x01_Socket, J8 Conn_01x01_Socket, J9 Barrel_Jack_Switch, P1 front_panel, P2 bottom_panel, Q1 MMBT5551, Q10 AO3401A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

Commit message: White pcbs.
Parts:
- removed BT1: Battery_Cell, pedale:BatteryHolder_Eagle_12BH611-GR, symbol Device:Battery_Cell
- removed J7, J8: Conn_01x01_Socket, TestPoint:TestPoint_THTPad_D2.5mm_Drill1.2mm, symbol Connector:Conn_01x01_Socket
- removed Q12: AO3400A, Package_TO_SOT_SMD:SOT-23, symbol Transistor_FET:AO3400A
- removed Q6: AO3401A, Package_TO_SOT_SMD:SOT-23, symbol Transistor_FET:AO3401A
- removed R23, R27: 100k, Resistor_SMD:R_0603_1608Metric_Pad0.98x0.95mm_HandSolder, symbol Device:R
- added J3, J4: Jack_6.35, pedale:Jack_6.35mm, symbol pedale:Jack_6.35
Connections:
- net 0: now also J3.S
- net IN_CONNECT: no longer names the net of J1.SN
- no-connect marks 11 -> 19
Other:
- title: Big Muff Pi -> Noise gate
